File: RT_PA_1_TSMC180.kicad_pcb (KiCad board)
At the start: 4 copper layers, 160 x 100 mm, 121 parts, among them J1 Conn_Coaxial, J10 Conn_01x01, J101 Conn_01x01, J11 Conn_01x01, J12 Conn_01x01, J13 Conn_01x01, J14 Conn_01x01_Female, J15 Conn_01x01_Female, J16 Conn_01x01, J171 Conn_01x01, J172 Conn_01x01, J173 Conn_01x01, J18 Conn_01x01, J19 Conn_01x01, J2 Conn_01x01, J20 Conn_01x01, J201 Conn_01x01, J202 Conn_01x01, J203 Conn_01x01, J22 Conn_01x01, J25 Conn_01x01, J27 Conn_01x01, J28 Conn_01x01, J29 Conn_Coaxial, J3 Conn_Coaxial, J31 Conn_Coaxial, J33 Conn_Coaxial, J35 Conn_Coaxial, J37 Conn_Coaxial, J39 Conn_Coaxial, J4 Conn_01x01, J401 Conn_01x02, J402 Conn_01x01, J41 Conn_Coaxial, J42 Conn_01x01, J43 Conn_Coaxial, J44 Conn_01x01, J45 Conn_01x01, J46 Conn_01x01, J47 Conn_01x01, J48 Conn_01x01, J49 Conn_01x04, J5 Conn_Coaxial, J50 Conn_01x04, J501 Conn_01x01, J51 Conn_01x01, J52 Conn_01x01, J53 Conn_01x01, J54 Conn_01x01, J55 Conn_01x02, J56 Conn_01x02, J57 Conn_01x02, J58 Conn_01x03, J6 Conn_01x01, J60 Conn_01x01, J61 Conn_01x02, J62 Conn_01x03, J63 Conn_01x01, J64 Conn_01x01, J65 Conn_Coaxial, J66 Conn_01x01, J67 Conn_Coaxial, J7 Conn_Coaxial, J8 Conn_01x01, J9 Conn_01x01_Female, U1 PART1p68

Commit message: Correction of the ASIC's symbole
Parts:
- added J17: Conn_01x01_Female, banana:Banana_test_point_4mm, F.Cu at (29.2, 81.3)
Connections:
- U1 pad 1: /VM_M -> /Vo1m
- U1 pad 2: /Vo1m -> /VM_M
- U1 pad 3: /VbiasO -> /pS
- U1 pad 4: /VbiasDiff -> /pB
- U1 pad 5: /VIbias -> /pG
- U1 pad 6: /VbiasM -> /pD
- U1 pad 63: GND -> /VDD_M
- U1 pad 64: /VDD_M -> GND
- U1 pad 65: /pD -> /VbiasM
- U1 pad 66: /pG -> /VIbias
- U1 pad 67: /pB -> /VbiasDiff
- U1 pad 68: /pS -> /VbiasO
- U1 pad 7: GND -> /VDD_M
- U1 pad 8: /VDD_M -> GND
